Commit message: Added Redundance Pose and Movement Finished Topic

File: iiwa_description/urdf/iiwa14.urdf.xacro (robot description, xacro)
@@ -10,5 +10,5 @@
   <xacro:arg name="origin_rpy" default="0 0 0"/>
   <!-- Fix to world just for testing -->
-  <link name="world"/>
+  <!--<link name="world"/>-->
   <!--iiwa-->
   <xacro:iiwa14 hardware_interface="$(arg hardware_interface)" robot_name="$(arg robot_name)" parent="world">
